Commit message: Chsnge package name to lower case letter

File: Manipulator_tf/urdf/Manipulator_tf.urdf (robot description, URDF)
Before this commit: robot Manipulator_tf, 8 links, 7 joints
Links:
- link arm_1_link: geometry collision mesh filename=package://manipulator_tf/meshes/arm_1_link.STL; visual mesh filename=package://manipulator_tf/meshes/arm_1_link.STL
- link arm_2_link: geometry collision mesh filename=package://manipulator_tf/meshes/arm_2_link.STL; visual mesh filename=package://manipulator_tf/meshes/arm_2_link.STL
- link arm_3_link: geometry collision mesh filename=package://manipulator_tf/meshes/arm_3_link.STL; visual mesh filename=package://manipulator_tf/meshes/arm_3_link.STL
- link arm_4_link: geometry collision mesh filename=package://manipulator_tf/meshes/arm_4_link.STL; visual mesh filename=package://manipulator_tf/meshes/arm_4_link.STL
- link arm_5_link: geometry collision mesh filename=package://manipulator_tf/meshes/arm_5_link.STL; visual mesh filename=package://manipulator_tf/meshes/arm_5_link.STL
- link arm_base_link: geometry collision mesh filename=package://manipulator_tf/meshes/arm_base_link.STL; visual mesh filename=package://manipulator_tf/meshes/arm_base_link.STL
- link base_link: geometry collision mesh filename=package://manipulator_tf/meshes/base_link.STL; visual mesh filename=package://manipulator_tf/meshes/base_link.STL
- link gripper_1_link: geometry collision mesh filename=package://manipulator_tf/meshes/gripper_1_link.STL; visual mesh filename=package://manipulator_tf/meshes/gripper_1_link.STL

Commit message: New tf file

File: Manipulator_tf/urdf/Manipulator_tf.urdf (robot description, URDF)
Before this commit: robot manipulator_tf, 8 links, 7 joints
Links:
- link base_link: mass 0.24083 -> 0.240825
Joints:
- joint arm_1_joint: origin xyz=0.12473 0.22085 0.24347 rpy=3.1416 1.1738 3.1416 -> xyz=0.124729378323661 0.220846589595659 0.24346647728671 rpy=3.14159265358979 1.17381591335885 3.14159265358979
- joint arm_2_joint: axis 0.38664 0 -0.92223 -> 0.386635347795088 0 -0.922232675540924; origin xyz=0.00057178 0.0325 0.00023971 rpy=0 0 0 -> xyz=0.000571784259143912 0.0325000000003336 0.000239713915762298 rpy=0 0 0
- joint arm_3_joint: axis 0.38664 0 -0.92223 -> 0.386635347795088 0 -0.922232675540924; origin xyz=0 0.152 0 rpy=0 0 0 -> xyz=0 0.151999999999983 0 rpy=0 0 0
- joint arm_4_joint: axis 0.38664 0 -0.92223 -> 0.386635347795096 0 -0.922232675540921; origin xyz=0 0.1464 0 rpy=0 0 0 -> xyz=0 0.146399999999996 0 rpy=0 0 0
- joint arm_5_joint: origin xyz=0.00056091 0.09115 0.0028104 rpy=3.1416 0 3.1416 -> xyz=0.000560909224782251 0.0911499999988545 0.00281042669964111 rpy=3.14159265358979 0 3.14159265358979
- joint arm_base_joint: origin xyz=-0.12473 0.24347 -0.18335 rpy=1.5708 0 0 -> xyz=-0.124729378323661 0.24346647728671 -0.183346589595995 rpy=1.5707963267949 0 0
