Commit message: Ik simple library
เขียน library สำหรับ IK ที่สามารถใช้งานได้

File: manipulator_tf2/urdf/manipulator_tf2.urdf (robot description, URDF)
Before this commit: robot manipulator_tf2, 8 links, 7 joints
Joints:
- joint arm_1_joint: type continuous -> revolute
- joint arm_2_joint: type continuous -> revolute
- joint arm_3_joint: type continuous -> revolute
- joint arm_4_joint: type continuous -> revolute
- joint arm_5_joint: type continuous -> revolute
- joint gripper_1_joint: type continuous -> revolute
